File: hardware/CC1125_Transceiver/_autosave-CC1125_Transceiver.kicad_pcb (KiCad board)
At the start: 2 copper layers, 29 parts, among them IC1 CC1125RHBT, IC2 GALI-74+

Commit message: updated
Parts:
- removed C1, C12: 47n, Capacitor_SMD:C_0402_1005Metric_Pad0.74x0.62mm_HandSolder
- added J1: SMA_Ant, Connector_Coaxial:SMA_Amphenol_132289_EdgeMount, F.Cu at (125.2, 64.0)
- added J2: Conn_02x05_Counter_Clockwise, Connector_PinSocket_2.54mm:PinSocket_2x05_P2.54mm_Vertical, F.Cu at (91.7, 58.1)
- added J3: Conn_01x05, Connector_PinHeader_2.54mm:PinHeader_1x05_P2.54mm_Horizontal, F.Cu at (78.6, 83.5)
- added L1: L, Inductor_SMD:L_0402_1005Metric_Pad0.77x0.64mm_HandSolder, F.Cu at (105.2, 66.2)
- added L2: L, Inductor_SMD:L_0402_1005Metric_Pad0.77x0.64mm_HandSolder, F.Cu at (107.0, 68.0)
- added L3: 39n, Inductor_SMD:L_0402_1005Metric_Pad0.77x0.64mm_HandSolder, F.Cu at (113.0, 62.6)
- added L4: L, Inductor_SMD:L_0402_1005Metric_Pad0.77x0.64mm_HandSolder, F.Cu at (120.6, 65.6)
- added L5: L, Inductor_SMD:L_0402_1005Metric_Pad0.77x0.64mm_HandSolder, F.Cu at (118.0, 65.6)
- added L6: 82n, Inductor_SMD:L_0402_1005Metric_Pad0.77x0.64mm_HandSolder, F.Cu at (110.6, 60.2)
- added L7: 82n, Inductor_SMD:L_0402_1005Metric_Pad0.77x0.64mm_HandSolder, F.Cu at (110.6, 62.6)
- added L8: 150n, Inductor_SMD:L_0402_1005Metric_Pad0.77x0.64mm_HandSolder, F.Cu at (108.6, 62.0)
- added L9: L, Inductor_SMD:L_0402_1005Metric_Pad0.77x0.64mm_HandSolder, F.Cu at (116.8, 70.2)
- added R1: R, Resistor_SMD:R_0402_1005Metric_Pad0.72x0.64mm_HandSolder, F.Cu at (104.8, 70.2)
- added R2: 28.7, Resistor_SMD:R_0402_1005Metric_Pad0.72x0.64mm_HandSolder, F.Cu at (119.4, 70.6)
- added REF**: ${Value}, libary:VHF_UHF_Module_generic, F.Cu at (112.0, 90.2)
- added REF**: H_Wurth_WE-SHC-SEAMLESS-FRAME_3670270, SHIELDING_SMD_Wurth:H_Wurth_WE-SHC-SEAMLESS-FRAME_3670270, F.Cu at (107.8, 63.4)
- C17: value 47n -> 100n
- moved C6 52.9 mm to (120.6, 64.0)
- moved C7 52.3 mm to (120.0, 67.6), turned to -90 degrees
- moved C10 49.2 mm to (119.4, 69.4), turned to 180 degrees
- moved C5 48.1 mm to (115.8, 63.6), turned to 135 degrees
- moved C11 46.1 mm to (116.8, 67.8), turned to 45 degrees
- moved C4 40.5 mm to (108.0, 67.0), turned to -45 degrees
- moved C9 40.0 mm to (110.6, 63.8)
- moved C8 39.9 mm to (110.6, 61.4)
- moved C2 39.5 mm to (105.8, 69.2), turned to 135 degrees
- moved C3 38.7 mm to (106.2, 65.2), turned to -45 degrees
- moved C21 33.8 mm to (106.2, 57.4), turned to 45 degrees
- moved R3 33.8 mm to (102.0, 67.8), turned to -90 degrees
- moved C19 33.4 mm to (107.0, 58.2), turned to 45 degrees
- moved C13 32.4 mm to (103.4, 66.8), turned to -90 degrees
- moved C22 30.5 mm to (107.8, 59.0), turned to 45 degrees
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Connections:
- C13 pad 1: Net-(IC1-AVDD_IF) -> +3V3
- C14 pad 1: Net-(IC1-AVDD_IF) -> +3V3
- C15 pad 1: Net-(IC1-AVDD_IF) -> +3V3
- C16 pad 1: Net-(IC1-AVDD_IF) -> +3V3
- C17 pad 1: Net-(IC1-AVDD_IF) -> +3V3
- C18 pad 1: Net-(IC1-AVDD_IF) -> +3V3
- C19 pad 1: Net-(IC1-AVDD_IF) -> +3V3
- C20 pad 1: Net-(IC1-AVDD_IF) -> +3V3
- IC1 pad 1: Net-(IC1-AVDD_IF) -> +3V3
- IC1 pad 10: unconnected-(IC1-GPIO0-Pad10) -> /GPIO
- IC1 pad 11: unconnected-(IC1-CSN-Pad11) -> /CSn
- IC1 pad 12: Net-(IC1-AVDD_IF) -> +3V3
- IC1 pad 13: Net-(IC1-AVDD_IF) -> +3V3
- IC1 pad 15: Net-(IC1-AVDD_IF) -> +3V3
- IC1 pad 2: unconnected-(IC1-RESET_N-Pad2) -> /Resetn
- IC1 pad 22: Net-(IC1-AVDD_IF) -> +3V3
- IC1 pad 25: Net-(IC1-AVDD_IF) -> +3V3
- IC1 pad 26: Net-(IC1-AVDD_IF) -> +3V3
- IC1 pad 27: Net-(IC1-AVDD_IF) -> +3V3
- IC1 pad 28: Net-(IC1-AVDD_IF) -> +3V3
- IC1 pad 3: unconnected-(IC1-GPIO3-Pad3) -> /GPI3
- IC1 pad 4: unconnected-(IC1-GPIO2-Pad4) -> /GPI2
- IC1 pad 5: Net-(IC1-AVDD_IF) -> +3V3
- IC1 pad 7: unconnected-(IC1-SI-Pad7) -> /SI
- IC1 pad 8: unconnected-(IC1-SCLK-Pad8) -> /SClk
- IC1 pad 9: unconnected-(IC1-SO(GPIO1)-Pad9) -> /SO
Routing:
- added copper zone on F.Cu, net GND
Other:
- board outline added: 43.8 x 18 mm
