File: hardware/CC1125_Transceiver/_autosave-CC1125_Transceiver.kicad_sch (KiCad schematic)
At the start: 44 parts, among them IC1 CC1125RHBT, IC2 GALI-74+, J1 SMA_Ant, J2 Conn_02x05_Counter_Clockwise, J3 Conn_01x05, Y1 40MHz

Commit message: updated
Parts:
- removed H1: 3670250, SHIELDING_SMD_Wurth:H_Wurth_WE-SHC-SEAMLESS-FRAME_3670250, symbol we_shield:3670250
- added H2: 3670288, libary:H_Wurth_WE-SHC-SEAMLESS-FRAME_3670288, symbol we_shield:3670288
Connections:
- net GND: now also H2.1 (GND)
Other:
- note added: "L8 bias current"
- note added: "TP?"
- note added: "TPD1E0B04?"
- note removed: "TP 2. Ordung"
