File: hardware/CC1125_Transceiver/CC1125_Transceiver.kicad_pcb (KiCad board)
At the start: 2 copper layers, 43.8 x 18 mm, 41 parts, among them IC1 CC1125RHBT, IC2 GALI-74+, J1 SMA_Ant, J2 Conn_02x05_Counter_Clockwise

Commit message: updated
Parts:
- added J3: Conn_01x05, Connector_PinHeader_2.54mm:PinHeader_1x05_P2.54mm_Horizontal, F.Cu at (78.6, 83.5)
- moved J1 2.49 mm to (127.6, 63.4)
- moved C10 2.00 mm to (119.4, 71.4)
- moved C13 0.89 mm to (103.0, 67.6)
- moved C5 0.81 mm to (115.0, 63.3), turned to 180 degrees
- moved C6 0.65 mm to (120.6, 63.4)
- moved L4 0.65 mm to (120.6, 65.0)
- moved L5 0.65 mm to (118.0, 65.0)
- moved C16 0.59 mm to (96.6, 61.6)
- moved C7 0.55 mm to (120.0, 67.0)
- moved C23 0.48 mm to (96.6, 62.8)
- moved C15 0.45 mm to (102.8, 56.4)
- moved C17 0.45 mm to (104.0, 56.4)
- moved C24 0.45 mm to (101.6, 56.4)
- moved C25 0.45 mm to (100.4, 56.4)
- moved C26 0.45 mm to (99.2, 56.4)
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Routing:
- net Net-(IC1-TRX_SW): track 0.00 -> 13.4 mm
- net Net-(D1-K): track 0.00 -> 7.67 mm
- net Net-(IC1-LNA_N): track 0.00 -> 7.64 mm
- net Net-(IC1-LNA_P): track 0.00 -> 7.50 mm
- net Net-(IC2-OUT&VCC): track 0.00 -> 5.65 mm
- net Net-(IC2-IN): track 0.00 -> 4.94 mm
- net Net-(C6-Pad1): track 0.00 -> 4.51 mm
- net Net-(IC1-PA): track 0.00 -> 3.97 mm
- net Net-(C2-Pad2): track 0.00 -> 3.79 mm
- net Net-(C8-Pad2): track 0.00 -> 3.69 mm
- net Net-(C3-Pad2): track 0.00 -> 2.83 mm
- net Net-(C11-Pad2): track 0.00 -> 2.26 mm
- net Net-(L9-Pad1): track 0.00 -> 1.43 mm
- net +3V3: track 0.00 -> 1.43 mm
- net +7V: track 0.00 -> 1.21 mm
Other:
- board size 43.8 x 18 mm -> 46 x 21.6 mm

Commit message: updated
Parts:
- removed J3: Conn_01x05, Connector_PinHeader_2.54mm:PinHeader_1x05_P2.54mm_Horizontal
- added Boot1: 434133025816, libary:434133025816, F.Cu at (96.0, 73.5)
- added C1: 100n, Capacitor_SMD:C_0402_1005Metric_Pad0.74x0.62mm_HandSolder, F.Cu at (91.8, 64.5)
- added C12: 100n, Capacitor_SMD:C_0402_1005Metric_Pad0.74x0.62mm_HandSolder, F.Cu at (85.3, 61.0)
- added C27: 1u, Capacitor_SMD:C_0402_1005Metric_Pad0.74x0.62mm_HandSolder, F.Cu at (81.6, 53.5)
- added C28: 4.7u|24V, Capacitor_SMD:C_0805_2012Metric_Pad1.18x1.45mm_HandSolder, F.Cu at (88.2, 53.7)
- added C29: 100n, Capacitor_SMD:C_0402_1005Metric_Pad0.74x0.62mm_HandSolder, F.Cu at (84.3, 53.5)
- added C30: 1u, Capacitor_SMD:C_0402_1005Metric_Pad0.74x0.62mm_HandSolder, F.Cu at (97.0, 69.4)
- added C31: 100n, Capacitor_SMD:C_0402_1005Metric_Pad0.74x0.62mm_HandSolder, F.Cu at (91.2, 70.2)
- added C32: 4.7u|24V, Capacitor_SMD:C_0805_2012Metric_Pad1.18x1.45mm_HandSolder, F.Cu at (92.0, 67.7)
- added C33: 100n, Capacitor_SMD:C_0402_1005Metric_Pad0.74x0.62mm_HandSolder, F.Cu at (99.5, 70.0)
- added C34: 100n, Capacitor_SMD:C_0402_1005Metric_Pad0.74x0.62mm_HandSolder, F.Cu at (94.5, 55.0)
- added C35: DNP, Capacitor_SMD:C_0402_1005Metric_Pad0.74x0.62mm_HandSolder, F.Cu at (92.0, 60.0)
- added D2: ~, LED_SMD:LED_0402_1005Metric_Pad0.77x0.64mm_HandSolder, F.Cu at (86.0, 69.5)
- added D3: ~, LED_SMD:LED_0402_1005Metric_Pad0.77x0.64mm_HandSolder, F.Cu at (88.0, 55.9)
- added H2: 3670288, libary:H_Wurth_WE-SHC-SEAMLESS-FRAME_3670290, F.Cu at (128.6, 93.8)
- added IC3: TLV61046ADBVT, libary:SOT95P280X145-6N, F.Cu at (83.7, 56.6)
- added IC4: TLV75801PDRVR, libary:SON65P200X200X80-7N, F.Cu at (96.3, 67.5)
- added J4: USB_C_Receptacle_USB2.0_14P, libary:USB421603A, F.Cu at (79.2, 65.7)
- added L10: 10uH/1A/190nO, libary:WE-TPC_282892, F.Cu at (79.8, 56.5)
- added R10: 10k, Resistor_SMD:R_0603_1608Metric_Pad0.98x0.95mm_HandSolder, F.Cu at (95.0, 64.7)
- added R11: 5.1k, Resistor_SMD:R_0402_1005Metric_Pad0.72x0.64mm_HandSolder, F.Cu at (88.5, 69.5)
- added R12: 5.1k, Resistor_SMD:R_0402_1005Metric_Pad0.72x0.64mm_HandSolder, F.Cu at (88.0, 58.5)
- added R13: 10k, Resistor_SMD:R_0603_1608Metric_Pad0.98x0.95mm_HandSolder, F.Cu at (96.8, 70.8)
- added R14: 10k, Resistor_SMD:R_0603_1608Metric_Pad0.98x0.95mm_HandSolder, F.Cu at (92.0, 58.5)
- added R4: 560k, Resistor_SMD:R_0402_1005Metric_Pad0.72x0.64mm_HandSolder, F.Cu at (86.8, 56.0)
- added R5: 71.5k, Resistor_SMD:R_0402_1005Metric_Pad0.72x0.64mm_HandSolder, F.Cu at (86.8, 58.5)
- added R6: 5.1k, Resistor_SMD:R_0603_1608Metric_Pad0.98x0.95mm_HandSolder, F.Cu at (84.0, 69.5)
- added R7: 5.1k, Resistor_SMD:R_0603_1608Metric_Pad0.98x0.95mm_HandSolder, F.Cu at (87.8, 71.0)
- added R8: 1M, Resistor_SMD:R_0402_1005Metric_Pad0.72x0.64mm_HandSolder, F.Cu at (93.9, 66.9)
- added R9: ToDo, Resistor_SMD:R_0402_1005Metric_Pad0.72x0.64mm_HandSolder, F.Cu at (94.6, 69.3)
- added Reset1: 434133025816, libary:434133025816, F.Cu at (88.5, 73.5)
- added U2: STM32L412K8Ux, Package_DFN_QFN:QFN-32-1EP_5x5mm_P0.5mm_EP3.45x3.45mm, F.Cu at (87.2, 64.8)
- added Y1: ECS-TXO-32CSMV-400-BN-TR, libary:ECSTXO32CSMV400BNTR, F.Cu at (92.0, 55.5)
- added Y2: 40MHz, libary:ABM8W480000MHZ6D1XT3, F.Cu at (98.5, 54.0)
- C11: value C -> 100n
- C14: value 47n -> 220n
- C17: value 100n -> 220n
- C3: value C -> 82p
- C4: value C -> 12p
- C6: value C -> 1.2p
- C7: value C -> 15p
- J2: value Conn_02x05_Counter_Clockwise -> Conn_02x03_Counter_Clockwise; footprint Connector_PinSocket_2.54mm:PinSocket_2x05_P2.54mm_Vertical -> Connector_PinHeader_1.00mm:PinHeader_2x03_P1.00mm_Vertical_SMD
- L2: value L -> 18n
- L4: value L -> 68n
- L5: value L -> 100n
- moved REF** 20.5 mm to (91.6, 91.2)
- moved J2 18.8 mm to (81.2, 73.8)
- moved C24 2.65 mm to (103.5, 54.5), turned to 0 degrees
- moved C16 1.63 mm to (95.0, 61.1)
- moved C23 1.63 mm to (95.0, 62.4)
- moved R2 1.40 mm to (118.0, 70.2), turned to -135 degrees
- moved C20 1.25 mm to (96.0, 58.5)
- moved C26 1.21 mm to (98.0, 56.5), turned to 0 degrees
- moved L9 0.73 mm to (117.0, 69.5), turned to 45 degrees
- moved C10 0.43 mm to (119.0, 71.2), turned to -135 degrees
- moved C25 0.18 mm to (100.5, 56.5), turned to 180 degrees
Connections:
- net /GPI2 renamed /CC_GPI2
- net /GPI3 renamed /CC_GPI3
- net /GPIO renamed /CC_GPIO
- net Net-(C11-Pad2) renamed /Filt2
- net Net-(D1-K) renamed /Anten
- net Net-(IC1-LNA_N) renamed /LNA_N
- net Net-(IC1-LNA_P) renamed /LNA_P
- net Net-(IC1-PA) renamed /PA1
- net Net-(IC1-TRX_SW) renamed /LNA_UB
- net Net-(IC2-IN) renamed /Filt1
- net Net-(IC2-OUT&VCC) renamed /PA2
- IC1 pad 11: /CSn -> /SPI_CSN
- IC1 pad 2: /Resetn -> /CC_Resetn
- IC1 pad 32: unconnected-(IC1-EXT_XOSC-Pad32) -> Net-(IC1-EXT_XOSC)
- IC1 pad 7: /SI -> /SPI_MOSI
- IC1 pad 8: /SClk -> /SPI_SCK
- IC1 pad 9: /SO -> /SPI_MISO
- J2 pad 1: unconnected-(J2-Pin_1-Pad1) -> /SPI_MOSI
- J2 pad 2: unconnected-(J2-Pin_2-Pad2) -> /CC_Resetn
- J2 pad 3: unconnected-(J2-Pin_3-Pad3) -> /SPI_SCK
- J2 pad 4: unconnected-(J2-Pin_4-Pad4) -> /SPI_MISO
- J2 pad 5: unconnected-(J2-Pin_5-Pad5) -> GND
- J2 pad 6: unconnected-(J2-Pin_6-Pad6) -> /SPI_CSN
Routing:
- net +3V3: track 1.43 -> 83.3 mm, vias 0 -> 16
- net +7V: track 1.21 -> 71.0 mm, vias 0 -> 2
- net VUSB: track 0.00 -> 60.1 mm, vias 0 -> 5
- net GND: track 0.00 -> 59.8 mm, vias 0 -> 72
- net /SPI_MOSI: track 0.00 -> 34.3 mm, vias 0 -> 2
- net /SPI_MISO: track 0.00 -> 33.2 mm, vias 0 -> 3
- net /SPI_SCK: track 0.00 -> 31.5 mm, vias 0 -> 2
- net /CC_Resetn: track 0.00 -> 24.5 mm, vias 0 -> 2
- net /SPI_CSN: track 0.00 -> 22.6 mm, vias 0 -> 2
- net /uc_Boot: track 0.00 -> 16.9 mm, vias 0 -> 2
- net /uc_Reset: track 0.00 -> 12.7 mm, vias 0 -> 2
- net Net-(IC1-EXT_XOSC): track 0.00 -> 11.8 mm
- net Net-(J4-CC2): track 0.00 -> 10.7 mm, vias 0 -> 2
- net Net-(J4-CC1): track 0.00 -> 9.12 mm, vias 0 -> 2
- net Net-(IC1-XOSC_Q1): track 0.00 -> 6.95 mm
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- added copper zone on In2.Cu, net +3V3
- added copper zone on B.Cu, net GND
- added copper zone on In1.Cu, net GND
- added copper zone on In2.Cu, net GND
Other:
- board size 46 x 21.6 mm -> 53.7 x 25.1 mm
- copper layers 2 -> 4
- board text added: "50Ω"
- board text added: "Sub GHz RF Transceiver"
- board text added: "V1.0 Fynn Gewiese"
- board text added: "boot"
- board text added: "reset"

Commit message: updated
Parts:
- removed REF**: ${Value}, libary:VHF_UHF_Module_generic
- added C36: DNP, Capacitor_SMD:C_0805_2012Metric_Pad1.18x1.45mm_HandSolder, B.Cu at (84.0, 96.0)
- added C37: DNP, Capacitor_SMD:C_0805_2012Metric_Pad1.18x1.45mm_HandSolder, B.Cu at (84.0, 99.5)
- added D4: ~, LED_SMD:LED_0402_1005Metric_Pad0.77x0.64mm_HandSolder, F.Cu at (89.0, 92.0)
- added R15: 5.1k, Resistor_SMD:R_0402_1005Metric_Pad0.72x0.64mm_HandSolder, F.Cu at (89.0, 89.5)
- added R16: 0, Resistor_SMD:R_0603_1608Metric_Pad0.98x0.95mm_HandSolder, B.Cu at (80.5, 97.5)
- H2: value 3670288 -> 3610637256S; footprint libary:H_Wurth_WE-SHC-SEAMLESS-FRAME_3670290 -> SHIELDING_SMD_Wurth:H_Wurth_WE-SHC-SMT-FRAME_3610637256S
- R6, R7: footprint Resistor_SMD:R_0603_1608Metric_Pad0.98x0.95mm_HandSolder -> Resistor_SMD:R_0402_1005Metric_Pad0.72x0.64mm_HandSolder
- moved R10 42.5 mm to (80.7, 104.6), turned to 0 degrees
- moved J1 38.5 mm to (141.6, 99.2)
- moved D3 36.1 mm to (87.5, 92.0)
- moved C31 35.2 mm to (83.7, 104.6)
- moved R13 35.1 mm to (87.7, 104.6)
- moved C33 35.0 mm to (88.3, 103.2), turned to 180 degrees
- moved Boot1 34.8 mm to (87.3, 107.2)
- moved C20 34.6 mm to (102.5, 92.5)
- moved Reset1 34.6 mm to (80.8, 107.2)
- moved C1 34.3 mm to (93.5, 98.8), turned to -90 degrees
- moved J2 33.8 mm to (92.5, 105.7), turned to 90 degrees
- moved C10 33.6 mm to (125.8, 104.2)
- moved C11 33.6 mm to (123.5, 100.7)
- moved C13 33.6 mm to (109.8, 100.5)
- moved C24 33.6 mm to (110.2, 87.4)
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Connections:
- D2 pad 1: Net-(D2-K) -> GND
- D2 pad 2: unconnected-(D2-A-Pad2) -> Net-(D2-A)
- D3 pad 1: Net-(D3-K) -> GND
- D3 pad 2: +7V -> Net-(D3-A)
- J4 pad A4: VUSB -> Net-(C37-Pad1)
- J4 pad B4: VUSB -> Net-(C37-Pad1)
- R11 pad 1: Net-(D2-K) -> unconnected-(R11-Pad1)
- R11 pad 2: GND -> Net-(D2-A)
- R12 pad 1: Net-(D3-K) -> +7V
- R12 pad 2: GND -> Net-(D3-A)
Routing:
- net +7V: track 71.0 -> 12.0 mm
- net +3V3: track 83.3 -> 26.8 mm, vias 16 -> 7
- net VUSB: track 60.1 -> 14.2 mm, vias 5 -> 3
- net GND: track 59.8 -> 18.7 mm, vias 72 -> 15
- net /SPI_MOSI: track 34.3 -> 6.21 mm, vias 2 -> 3
- net /SPI_MISO: track 33.2 -> 5.75 mm
- net /SPI_SCK: track 31.5 -> 4.75 mm, vias 2 -> 3
- net /CC_Resetn: track 24.5 -> 3.40 mm
- net /SPI_CSN: track 22.6 -> 6.30 mm
- net Net-(C37-Pad1): track 0.00 -> 12.3 mm, vias 0 -> 1
- net Net-(IC1-EXT_XOSC): track 11.8 -> 0.00 mm
- net /uc_Reset: track 12.7 -> 2.05 mm, vias 2 -> 1
- net /uc_Boot: track 16.9 -> 6.76 mm, vias 2 -> 0
- net Net-(J4-CC2): track 10.7 -> 2.14 mm, vias 2 -> 0
- net Net-(J4-CC1): track 9.12 -> 1.98 mm, vias 2 -> 0
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- removed copper zone on In2.Cu, net +3V3
Other:
- board size 53.7 x 25.1 mm -> 67 x 28.8 mm
- board text added: "<GHz Trans ceiver"
- board text added: "PA"
- board text added: "V1.0 Gewiese"
- board text added: "VCC"
- board text added: "rst"
- board text added: "uC"
- board text removed: "50Ω"
- board text removed: "Sub GHz RF Transceiver"
- board text removed: "V1.0 Fynn Gewiese"
- board text removed: "reset"

Commit message: updated
Routing:
- net +7V: track 12.0 -> 16.7 mm
Changed lines of the file:
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@@
 		(layer "F.Mask")
+	)
+	(gr_rect
+		(start 112.5 87)
+		(end 137.5 107)
+		(stroke
+			(width 0.2)
+			(type default)
+		)
+		(fill yes)
+		(layer "B.Mask")
 	)
 	(gr_arc
@@
 	)
 	(gr_text "\n<GHz\nTrans\nceiver"
-		(at 138.5 91 0)
+		(at 138.55 90.05 0)
 		(layer "F.Mask" knockout)
 		(effects
@@
 	)
 	(segment
+		(start 111.974265 93.474265)
+		(end 111.69853 93.75)
+		(width 0.2)
+		(layer "F.Cu")
+		(net 3)
+	)
+	(segment
 		(start 93.005 97.6875)
 		(end 93.5 98.1825)
@@
 	)
 	(segment
-		(start 113.698717 91.451283)
-		(end 113.698717 91.749813)
-		(width 0.2)
-		(layer "F.Cu")
-		(net 3)
-	)
-	(segment
 		(start 109.95 92.05)
 		(end 109.95 91.25)
@@
 	)
 	(segment
+		(start 111.69853 93.75)
+		(end 110.65 93.75)
+		(width 0.2)
+		(layer "F.Cu")
+		(net 3)
+	)
+	(segment
+		(start 113.698717 91.749813)
+		(end 113.698717 91.451283)
+		(width 0.2)
+		(layer "F.Cu")
+		(net 3)
+	)
+	(segment
 		(start 109.6 90.6)
 		(end 109.3 90.9)
@@
 	)
 	(segment
-		(start 110.65 93.75)
-		(end 111.69853 93.75)
-		(width 0.2)
-		(layer "F.Cu")
-		(net 3)
-	)
-	(segment
 		(start 108.45 91.75)
 		(end 109.3 90.9)
@@
 	)
 	(segment
+		(start 111.974265 93.474265)
+		(end 113.698717 91.749813)
+		(width 0.2)
+		(layer "F.Cu")
+		(net 3)
+	)
+	(segment
 		(start 90.9375 97.6875)
 		(end 93.005 97.6875)
@@
 		(start 110.8 89.8175)
 		(end 110.8 90.4)
-		(width 0.2)
-		(layer "F.Cu")
-		(net 3)
-	)
-	(segment
-		(start 111.69853 93.75)
-		(end 112.924265 92.524265)
-		(width 0.2)
-		(layer "F.Cu")
-		(net 3)
-	)
-	(segment
-		(start 113.698717 91.749813)
-		(end 112.924265 92.524265)
 		(width 0.2)
 		(layer "F.Cu")
@@
 	)
 	(via
-		(at 112.924265 92.524265)
+		(at 111.974265 93.474265)
 		(size 0.6)
 		(drill 0.3)
@@
 	)
 	(segment
+		(start 124 108.5)
+		(end 126.65 105.85)
+		(width 0.2)
+		(layer "F.Cu")
+		(net 8)
+	)
+	(segment
 		(start 85.9575 85.16)
 		(end 86.369 84.7485)
@@
 	)
 	(segment
-		(start 127.102566 104.65)
+		(start 126.65 104.197434)
 		(end 126.201283 103.748717)
 		(width 0.2)
@@
 	)
 	(segment
+		(start 126.65 105.85)
+		(end 126.65 104.197434)
+		(width 0.2)
+		(layer "F.Cu")
+		(net 8)
+	)
+	(segment
 		(start 125.222496 102.76993)
 		(end 126.201283 103.748717)
@@
 	)
 	(via
-		(at 127.102566 104.65)
+		(at 124 108.5)
 		(size 0.6)
 		(drill 0.3)
