File: hardware/CC1125_Transceiver/CC1125_Transceiver.kicad_sch (KiCad schematic)
At the start: 43 parts, among them IC1 CC1125RHBT, IC2 GALI-74+, J1 SMA_Ant, Y1 40MHz

Commit message: updated
Parts:
- removed C1, C12: 47n, Capacitor_SMD:C_0402_1005Metric_Pad0.74x0.62mm_HandSolder, symbol Device:C_Small
- added H1: 3670250, SHIELDING_SMD_Wurth:H_Wurth_WE-SHC-SEAMLESS-FRAME_3670250, symbol we_shield:3670250
- added J2: Conn_02x05_Counter_Clockwise, Connector_PinSocket_2.54mm:PinSocket_2x05_P2.54mm_Vertical, symbol Connector_Generic:Conn_02x05_Counter_Clockwise
- added J3: Conn_01x05, Connector_PinHeader_2.54mm:PinHeader_1x05_P2.54mm_Horizontal, symbol Connector:Conn_01x05_Pin
- C17: value 47n -> 100n
- IC1: footprint QFN50P500X500X100-33N-D -> (none)
- IC2: footprint GVA63 -> libary:GVA63
- J1: footprint (none) -> Connector_Coaxial:SMA_Amphenol_132289_EdgeMount
- L1, L2, L3, L4, L5, L6, L7, L8, L9: footprint (none) -> Inductor_SMD:L_0402_1005Metric_Pad0.77x0.64mm_HandSolder
- R1, R2: footprint (none) -> Resistor_SMD:R_0402_1005Metric_Pad0.72x0.64mm_HandSolder
Connections:
- net +3V3: now also C13.1, C14.1, C15.1, C16.1, C17.1, C18.1, C19.1, C20.1, IC1.1 (VDD_GUARD), IC1.12 (DVDD_2), IC1.13 (AVDD_IF), IC1.15 (AVDD_RF), IC1.22 (AVDD_SYNTH1), IC1.25 (AVDD_PFD_CHP), IC1.26 (DCPL_PFD_CHP), IC1.27 (AVDD_SYNTH2), IC1.28 (AVDD_XOSC), IC1.5 (DVDD_1)
- net GPIO: now reaches IC1.10 (GPIO0)
- net CSn: now reaches IC1.11 (CSN)
- net Resetn: now reaches IC1.2 (RESET_N)
- net GPI3: now reaches IC1.3 (GPIO3)
- net GPI2: now reaches IC1.4 (GPIO2)
- net SI: now reaches IC1.7 (SI)
- net SClk: now reaches IC1.8 (SCLK)
- net SO: now reaches IC1.9 (SO(GPIO1))
Other:
- moved on the sheet: C13, C15, C16, C17, C18, C19, C20

Commit message: updated
Parts:
- removed H1: 3670250, SHIELDING_SMD_Wurth:H_Wurth_WE-SHC-SEAMLESS-FRAME_3670250, symbol we_shield:3670250
- added H2: 3670288, libary:H_Wurth_WE-SHC-SEAMLESS-FRAME_3670288, symbol we_shield:3670288
Connections:
- net GND: now also H2.1 (GND)

Commit message: updated
Parts:
- removed J2: Conn_02x05_Counter_Clockwise, Connector_PinSocket_2.54mm:PinSocket_2x05_P2.54mm_Vertical, symbol Connector_Generic:Conn_02x05_Counter_Clockwise
- removed J3: Conn_01x05, Connector_PinHeader_2.54mm:PinHeader_1x05_P2.54mm_Horizontal, symbol Connector:Conn_01x05_Pin
- removed Y1: 40MHz, symbol Device:Crystal_Small
- added Boot1, Reset1: 434133025816, libary:434133025816, symbol libary:SW_Push_Shielded
- added C1, C12, C29, C31, C33, C34: 100n, Capacitor_SMD:C_0402_1005Metric_Pad0.74x0.62mm_HandSolder, symbol Device:C_Small
- added C27, C30: 1u, Capacitor_SMD:C_0402_1005Metric_Pad0.74x0.62mm_HandSolder, symbol Device:C_Small
- added C28, C32: 4.7u|24V, Capacitor_SMD:C_0805_2012Metric_Pad1.18x1.45mm_HandSolder, symbol Device:C_Small
- added C35: DNP, Capacitor_SMD:C_0402_1005Metric_Pad0.74x0.62mm_HandSolder, symbol Device:C_Small
- added D2, D3: ~, LED_SMD:LED_0402_1005Metric_Pad0.77x0.64mm_HandSolder, symbol Device:LED_Small
- added IC3: TLV61046ADBVT, libary:SOT95P280X145-6N, symbol libary:TLV61046ADBVT
- added IC4: TLV75801PDRVR, libary:SON65P200X200X80-7N, symbol libary:TLV75801PDRVR
- added J2: Conn_02x03_Counter_Clockwise, PinHeader_2x03_P1.00mm_Vertical_SMD, symbol Connector_Generic:Conn_02x03_Odd_Even
- added J4: USB_C_Receptacle_USB2.0_14P, libary:USB421603A, symbol Connector:USB_C_Receptacle_USB2.0_14P
- added L10: 10uH/1A/190nO, libary:WE-TPC_282892, symbol Device:L_Iron_Small
- added R10, R13, R14: 10k, Resistor_SMD:R_0603_1608Metric_Pad0.98x0.95mm_HandSolder, symbol Device:R_Small
- added R11, R12: 5.1k, Resistor_SMD:R_0402_1005Metric_Pad0.72x0.64mm_HandSolder, symbol Device:R_Small
- added R4: 560k, Resistor_SMD:R_0402_1005Metric_Pad0.72x0.64mm_HandSolder, symbol Device:R_Small
- added R5: 71.5k, Resistor_SMD:R_0402_1005Metric_Pad0.72x0.64mm_HandSolder, symbol Device:R_Small
- added R6, R7: 5.1k, Resistor_SMD:R_0603_1608Metric_Pad0.98x0.95mm_HandSolder, symbol Device:R_Small
- added R8: 1M, Resistor_SMD:R_0402_1005Metric_Pad0.72x0.64mm_HandSolder, symbol Device:R_Small
- added R9: ToDo, Resistor_SMD:R_0402_1005Metric_Pad0.72x0.64mm_HandSolder, symbol Device:R_Small
- added U2: STM32L412K8Ux, Package_DFN_QFN:QFN-32-1EP_5x5mm_P0.5mm_EP3.45x3.45mm, symbol MCU_ST_STM32L4:STM32L412K8Ux
- added V1, V2, V3, V4: VSIN, symbol Simulation_SPICE:VSIN
- added Y1: ECS-TXO-32CSMV-400-BN-TR, ECSTXO32CSMV400BNTR, symbol libary:ECS-TXO-32CSMV-400-BN-TR
- added Y2: 40MHz, libary:ABM8W480000MHZ6D1XT3, symbol Device:Crystal_GND2
- C11: value C -> 100n
- C14: value 47n -> 220n
- C17: value 100n -> 220n
- C3: value C -> 82p
- C4: value C -> 12p
- C6: value C -> 1.2p
- C7: value C -> 15p
- H2: footprint libary:H_Wurth_WE-SHC-SEAMLESS-FRAME_3670288 -> libary:H_Wurth_WE-SHC-SEAMLESS-FRAME_3670290
- IC1: footprint (none) -> libary:QFN50P500X500X100-33N-D
- L2: value L -> 18n
- L4: value L -> 68n
- L5: value L -> 100n
Connections:
- net +3V3: now also Boot1.1, C1.1, C12.1, C32.1, C34.1, IC4.1 (OUT), R10.1, R8.1, U2.1 (VDD), U2.17 (VDD), U2.5 (VDDA), Y1.4 (VDD)
- net +7V: now also C28.1, C29.1, D3.2 (A), IC3.5 (VOUT), R4.1
- net GND: now also Boot1.SH (B), C1.2, C12.2, C27.2, C28.2, C29.2, C30.2, C31.2, C32.2, C33.2, C34.2, C35.2, IC3.2 (GND), IC4.3 (GND), IC4.7 (EP), J2.5 (Pin_5), J4.A1 (GND), J4.A12 (GND), J4.B1 (GND), J4.B12 (GND), J4.S1 (SHIELD), R11.2, R12.2, R13.2, R14.2, R5.2, R6.2, R7.2, R9.2, Reset1.1, Reset1.SH (B), U2.16 (VSS), U2.32 (VSS), U2.33 (VSS), V2.2, V3.2, V4.2, Y1.1 (GND), Y1.2 (GND), Y2.2
- net PA2: now reaches C11.1, IC2.3 (OUT&VCC), L9.2
- net LNA_N: now reaches C8.1, IC1.20 (LNA_N), L6.1, L8.2
- net LNA_N: now also V1.2
- net Filt2: now reaches C11.2, C5.1, L5.1
- net LNA_UB: now reaches C5.2, IC1.18 (TRX_SW), L3.2
- net LNA_UB: now also V3.1
- net Anten: now reaches C6.2, D1.1 (K), J1.1 (In), L4.2
- net Anten: now also V2.1
- net LNA_P: now reaches C9.1, IC1.19 (LNA_P), L7.1, L8.1
- net LNA_P: now also V1.1
- net at C26.1, IC1.31 (XOSC_Q2): now also Y2.3
- net at C25.1, IC1.30 (XOSC_Q1): now also Y2.1
- net PA1: now reaches C3.1, IC1.17 (PA), L1.2
- net PA1: now also V4.1
- net Filt1: now reaches C4.2, IC2.1 (IN), L2.2
- net at IC1.32 (EXT_XOSC): now also C35.1, R14.1, Y1.3 (OUT)
- net CSn renamed SPI_CSN
- net SPI_CSN: now also J2.6 (Pin_6)
- net GPI2 renamed CC_GPI2
- net GPI3 renamed CC_GPI3
- net GPIO renamed CC_GPIO
- net Resetn renamed CC_Resetn
- net CC_Resetn: now also J2.2 (Pin_2)
- net SClk renamed SPI_SCK
- net SPI_SCK: now also J2.3 (Pin_3), U2.7 (PA1)
- net SI renamed SPI_MOSI
- net SPI_MOSI: now also J2.1 (Pin_1), U2.13 (PA7)
- net SO renamed SPI_MISO
- net SPI_MISO: now also J2.4 (Pin_4), U2.12 (PA6)
- new net: J4.A5 (CC1), R6.1
- new net: J4.B5 (CC2), R7.1
- new net: IC3.1 (SW), L10.2
- new net: IC3.3 (FB), R4.2, R5.1
- new net: D3.1 (K), R12.1
- new net: IC4.2 (FB), R8.2, R9.1
- new net: D2.1 (K), R11.1
- new net USB_DN: J4.A7 (D-), J4.B7 (D-), U2.21 (PA11)
- new net USB_DP: J4.A6 (D+), J4.B6 (D+), U2.22 (PA12)
- new net VUSB: C27.1, C30.1, IC3.4 (EN), IC3.6 (VIN), IC4.4 (EN), IC4.6 (IN), J4.A4 (VBUS), J4.A9 (VBUS), J4.B4 (VBUS), J4.B9 (VBUS), L10.1
- new net uc_Boot: Boot1.2, C33.1, R13.1, U2.31 (PH3)
- new net uc_Reset: C31.1, R10.2, Reset1.2, U2.4 (NRST)
Other:
- note added: "ABM8W-40.0000MHZ-4-B1U-T3"
- note added: "VFB = 0.55 V"
- note added: "VOUT = VFB × (1 + R1 / R2)"
- moved on the sheet: C13, C14, C16

Commit message: updated
Parts:
- added C36, C37: DNP, Capacitor_SMD:C_0805_2012Metric_Pad1.18x1.45mm_HandSolder, symbol Device:C_Small
- added C38: 220n, Capacitor_SMD:C_0402_1005Metric_Pad0.74x0.62mm_HandSolder, symbol Device:C_Small
- added D4: ~, LED_SMD:LED_0402_1005Metric_Pad0.77x0.64mm_HandSolder, symbol Device:LED_Small
- added R15: 5.1k, Resistor_SMD:R_0402_1005Metric_Pad0.72x0.64mm_HandSolder, symbol Device:R_Small
- added R16: 0, Resistor_SMD:R_0603_1608Metric_Pad0.98x0.95mm_HandSolder, symbol Device:R_Small
- H2: value 3670288 -> 3610637256S; footprint libary:H_Wurth_WE-SHC-SEAMLESS-FRAME_3670290 -> SHIELDING_SMD_Wurth:H_Wurth_WE-SHC-SMT-FRAME_3610637256S
- IC1: footprint libary:QFN50P500X500X100-33N-D -> QFN50P500X500X100-33N-D
- R6, R7: footprint Resistor_SMD:R_0603_1608Metric_Pad0.98x0.95mm_HandSolder -> Resistor_SMD:R_0402_1005Metric_Pad0.72x0.64mm_HandSolder
Connections:
- net +3V3: now also R15.1; no longer IC1.26 (DCPL_PFD_CHP)
- net +7V: now also R12.1; no longer D3.2 (A)
- net GND: now also D2.1 (K), D3.1 (K), C36.2, C37.2, C38.2, D4.1 (K); no longer R11.2, R12.2
- net VUSB: now also C36.1, R16.2; no longer J4.A4 (VBUS), J4.A9 (VBUS), J4.B4 (VBUS), J4.B9 (VBUS)
- net at R11.1: no longer D2.1 (K)
- net at D2.2 (A): now also R11.2
- net Filt2 renamed Rx/Tx
- new net: C38.1, IC1.26 (DCPL_PFD_CHP)
- new net: D4.2 (A), R15.2
- new net: C37.1, J4.A4 (VBUS), J4.A9 (VBUS), J4.B4 (VBUS), J4.B9 (VBUS), R16.1
- new net: D3.2 (A), R12.2
Other:
- note added: "ESD necessary or DC Block caps enough? SAW Filter?"
- note added: "Simulation"
- note removed: "ESD necessary or DC Block caps enough?"
- moved on the sheet: C22, C23, C24, D1, D2, D3, J1, J4, R11, R12, R6, R7
